File: pcbs/jabr-control-v1/jabr-control-v1.kicad_pcb (KiCad board)
At the start: 6 copper layers, 70 x 80 mm, 183 parts, among them J10001 ARJM11D7-502-AB-EW2, J10002 TYPE-C-31-M-12, J4001 MDT320E0X001, J401 U.FL-R-SMT-K_895, J402 U.FL-R-SMT-K_895, J6001 MSPE-J2L0-x00, J9001 43045-0201, Q2602 DMN21D2UFB-7B, U1201 TPS259472ARPWR, U1301 MAX20004AFOC/VY+T, U1501 TPS62290TDRVRQ1, U2401 PESD4USB3BTTS-QX, U2402 PESD4USB3BTTS-QX, U301 TVS3301DRBR, U302 TPS26600RHFR, U303 PI7C9X2G304SL, U3801 TPS62290TDRVRQ1, U401 LMQ66430MC3RXBRQ1, U402 TPS7B8133QDRVRQ1, U403 TPS2116DRL, U5001 LAN7431_YXX, U8001 LAN8870, Y401 ASEK-32.768KHZ-LRT, Y8001 XRCGB25M000F3A16R0

Commit message: Schematic nearing completion, need to do GPIO and PHY decouplings caps
Parts:
- removed TP2001, TP2002: 1.5mm, TestPoint:TestPoint_Pad_D1.5mm
- added C1001: 4u7, project_footprints:C_0402, F.Cu at (105.4, 77.5)
- added C1002: 4u7, project_footprints:C_0402, F.Cu at (105.4, 79.4)
- added C1003: 4u7, project_footprints:C_0402, F.Cu at (105.4, 81.4)
- added C1004: 4u7, project_footprints:C_0402, F.Cu at (105.4, 83.4)
- added C1409: 4u7, project_footprints:C_0402, F.Cu at (69.7, 89.3)
- added C1410: 4u7, project_footprints:C_0402, F.Cu at (72.5, 77.5)
- added C1411: 22p, project_footprints:C_0402, F.Cu at (72.5, 79.4)
- added C1412: 4u7, project_footprints:C_0402, F.Cu at (72.5, 81.4)
- added C1413: 4u7, project_footprints:C_0402, F.Cu at (72.5, 83.4)
- added C1414: 4u7, project_footprints:C_0402, F.Cu at (72.5, 85.3)
- added C1507: 4u7, project_footprints:C_0402, F.Cu at (116.7, 88.5)
- added C1508: 4u7, project_footprints:C_0402, F.Cu at (116.7, 90.5)
- added C303: 4u7, project_footprints:C_0402, F.Cu at (66.8, 97.7)
- added C304: 100n, project_footprints:C_0402, F.Cu at (66.8, 99.7)
- added C305: 100n, project_footprints:C_0402, F.Cu at (66.8, 101.7)
- added C306: 100n, project_footprints:C_0402, F.Cu at (66.8, 103.6)
- added C307: 100n, project_footprints:C_0402, F.Cu at (66.8, 105.6)
- added C308: 100n, project_footprints:C_0402, F.Cu at (66.8, 107.6)
- added C309: 100n, project_footprints:C_0402, F.Cu at (66.8, 109.5)
- added C310: 100n, project_footprints:C_0402, F.Cu at (66.8, 111.5)
- added C311: 100n, project_footprints:C_0402, F.Cu at (69.7, 97.7)
- added C312: 100n, project_footprints:C_0402, F.Cu at (69.7, 99.7)
- added C313: 100n, project_footprints:C_0402, F.Cu at (69.7, 101.7)
- added C314: 4u7, project_footprints:C_0402, F.Cu at (69.7, 103.6)
- added C315: 100n, project_footprints:C_0402, F.Cu at (69.7, 105.6)
- added C316: 100n, project_footprints:C_0402, F.Cu at (69.7, 107.6)
- added C317: 100n, project_footprints:C_0402, F.Cu at (69.7, 109.5)
- added C318: 100n, project_footprints:C_0402, F.Cu at (69.7, 111.5)
- added C319: 100n, project_footprints:C_0402, F.Cu at (72.5, 97.7)
- added C320: 100n, project_footprints:C_0402, F.Cu at (72.5, 99.7)
- added C321: 100n, project_footprints:C_0402, F.Cu at (72.5, 101.7)
- added C322: 100n, project_footprints:C_0402, F.Cu at (72.5, 103.6)
- added C323: 100n, project_footprints:C_0402, F.Cu at (72.5, 105.6)
- added C324: 100n, project_footprints:C_0402, F.Cu at (72.5, 107.6)
- added C325: 100n, project_footprints:C_0402, F.Cu at (72.5, 109.5)
- added C326: 100n, project_footprints:C_0402, F.Cu at (72.5, 111.5)
- added C327: 100n, project_footprints:C_0402, F.Cu at (75.4, 97.7)
- added C328: 100n, project_footprints:C_0402, F.Cu at (75.4, 99.7)
- added C329: 100n, project_footprints:C_0402, F.Cu at (75.4, 101.7)
- added C330: 100n, project_footprints:C_0402, F.Cu at (75.4, 103.6)
- added C331: 4u7, project_footprints:C_0402, F.Cu at (75.4, 105.6)
- added D1001: SZESD8472MUT5G, project_footprints:SZESD7462N2T5G, F.Cu at (105.4, 90.9)
- added D1002: SZESD8472MUT5G, project_footprints:SZESD7462N2T5G, F.Cu at (105.4, 93.0)
- added J1001: 48406-0003, project_footprints:48406-0003, F.Cu at (162.5, 136.5)
- added J201: JST-SH-4-Vertical, project_footprints:JST_SH_BM04B-SRSS-TB_1x04-1MP_P1.00mm_Vertical, F.Cu at (175.0, 75.5)
- added L1401: 78438313015, project_footprints:L_Wurth_WE-MAIA-1610, F.Cu at (82.1, 84.9)
- added R1401: 810k, project_footprints:R_0402, F.Cu at (79.0, 81.5)
- added R1402: 180k, project_footprints:R_0402, F.Cu at (79.0, 83.5)
- added R202: 10k, project_footprints:R_0402, F.Cu at (109.4, 106.0)
- added R305: 10k, project_footprints:R_0402, F.Cu at (81.2, 108.4)
- added S201: PCM12SMTBR, project_footprints:PCM12SMTBR, B.Cu at (132.0, 107.5)
- added SW202: TS20-42-25-WT-160-SMT-TR, project_footprints:TS204225WT160SMTTR, F.Cu at (195.0, 73.5)
- added TP1402: 1.5mm, project_footprints:TestPoint_Pad_D1.5mm, F.Cu at (75.8, 85.4)
- added TP201: 1.5mm, project_footprints:TestPoint_Pad_D1.5mm, F.Cu at (106.1, 98.5)
- added TP202: 1.5mm, project_footprints:TestPoint_Pad_D1.5mm, F.Cu at (106.1, 102.0)
- added TP203: 1.5mm, project_footprints:TestPoint_Pad_D1.5mm, F.Cu at (106.1, 105.6)
- added TP204: 1.5mm, project_footprints:TestPoint_Pad_D1.5mm, F.Cu at (106.1, 109.2)
- added U1001: AP22653FDZ-7, project_footprints:SON65P200X200X80-7N-D, F.Cu at (106.2, 88.1)
- added U1002: PESD4USB3BTTS-QX, project_footprints:PESD4USB3BTTSQX, F.Cu at (102.0, 77.9)
- added U1003: PESD4USB3BTTS-QX, project_footprints:PESD4USB3BTTSQX, F.Cu at (102.0, 80.9)
- added U1004: PESD4USB3BTTS-QX, project_footprints:PESD4USB3BTTSQX, F.Cu at (102.0, 84.0)
- added U1005: PESD4USB3BTTS-QX, project_footprints:PESD4USB3BTTSQX, F.Cu at (102.0, 87.0)
- added U1401: TPS62290TDRVRQ1, project_footprints:SON65P200X200X80-7N, F.Cu at (82.4, 81.6)
- added U201: NX3DV221TKX, project_footprints:SON50P300X300X100-11N, F.Cu at (166.0, 124.5)
- C1301, C1302, C1309, C1310, C1311, C401, C402: footprint Capacitor_SMD:C_0805_2012Metric -> project_footprints:C_0805
- C2401, C403, C404, C405, C406, C407: footprint Capacitor_SMD:C_0402_1005Metric -> project_footprints:C_0402
- C301, C302, C601: footprint Capacitor_SMD:C_0603_1608Metric -> project_footprints:C_0603
- R301, R302, R303, R304, R402, R403: footprint Resistor_SMD:R_0402_1005Metric -> project_footprints:R_0402
- TP1301, TP1401, TP1501, TP301, TP302, TP303, TP3801, TP401, TP8001, TP8002, TP801: footprint TestPoint:TestPoint_Pad_D1.5mm -> project_footprints:TestPoint_Pad_D1.5mm
- moved U2402 107.4 mm to (102.0, 93.0)
- moved U2401 107.2 mm to (102.0, 90.0)
- moved C1403 100.8 mm to (69.7, 77.5)
- moved C1404 100.8 mm to (69.7, 79.4)
- moved C1405 100.8 mm to (69.7, 81.4)
- moved C1406 100.8 mm to (69.7, 83.4)
- moved C1407 100.8 mm to (69.7, 85.3)
- moved C1408 100.8 mm to (69.7, 87.3)
- moved D303 100.4 mm to (117.0, 77.8)
- moved D302 100.3 mm to (115.7, 81.6)
- moved D601 100.3 mm to (115.7, 83.6)
- moved D301 98.2 mm to (96.8, 80.0)
- moved FL301 96.5 mm to (113.0, 78.5)
- moved Y8001 93.3 mm to (76.7, 125.1)
- moved TP1401 92.8 mm to (75.8, 81.8)
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Connections:
- net /CM5/~{BT_DISABLE} renamed /CM5/BT_EN
- net /CM5/~{WL_DISABLE} renamed /CM5/WL_EN
- C502 pad 1: +3V3 -> +3V3_PCIE
- C526 pad 1: +3V3 -> +3V3_PCIE
- J10001 pad 11: unconnected-(J10001-ANODE-Pad11) -> +3V3
- J10001 pad 12: unconnected-(J10001-CATHODE-Pad12) -> /CM5IO/LEDG
- J10001 pad 13: unconnected-(J10001-ANODE-Pad13) -> +3V3
- J10001 pad 14: unconnected-(J10001-CATHODE-Pad14) -> /CM5IO/LEDY
- J10001 pad 15: unconnected-(J10001-SHIELD-Pad15) -> GND
- J10001 pad 16: unconnected-(J10001-SHIELD-Pad16) -> GND
- J10002 pad A1_B12: Net-(J10002-GND-PadA1_B12) -> GND
- J10002 pad A4_B9: Net-(J10002-VBUS-PadA4_B9) -> VBUS
- J10002 pad A5: unconnected-(J10002-CC1-PadA5) -> /CM5/USB2_DEV.CC1
- J10002 pad A6: unconnected-(J10002-DP1-PadA6) -> /CM5/USB2_DEV.DP
- J10002 pad A7: unconnected-(J10002-DN1-PadA7) -> /CM5/USB2_DEV.DN
- J10002 pad B1_A12: Net-(J10002-GND-PadA1_B12) -> GND
- J10002 pad B4_A9: Net-(J10002-VBUS-PadA4_B9) -> VBUS
- J10002 pad B5: unconnected-(J10002-CC2-PadB5) -> /CM5/USB2_DEV.CC2
- J10002 pad B6: unconnected-(J10002-DP2-PadB6) -> /CM5/USB2_DEV.DP
- J10002 pad B7: unconnected-(J10002-DN2-PadB7) -> /CM5/USB2_DEV.DN
- J10002 pad S1: unconnected-(J10002-SHIELD-PadS1) -> GND
- J10002 pad S2: unconnected-(J10002-SHIELD-PadS2) -> GND
- J10002 pad S3: unconnected-(J10002-SHIELD-PadS3) -> GND
- J10002 pad S4: unconnected-(J10002-SHIELD-PadS4) -> GND
- J4001 pad 3: /M.2 E-Key/USB.DP -> /CM5/USB2_HOST.DP
- J4001 pad 5: /M.2 E-Key/USB.DN -> /CM5/USB2_HOST.DN
- SOM2001 pad 100: unconnected-(SOM2001C-CAM_GPIO1-Pad100) -> /CM5/CAM_GPIO1
- SOM2001 pad 101: /CM5/USB_OTG_ID -> GND
- SOM2001 pad 103: /CM5/USB.DN -> /CM5/DN
- SOM2001 pad 105: /CM5/USB.DP -> /CM5/DP
- SOM2001 pad 115: unconnected-(SOM2001C-MIPI0_D0_N-Pad115) -> /CM5/MIPI0.D0_N
- SOM2001 pad 117: unconnected-(SOM2001C-MIPI0_D0_P-Pad117) -> /CM5/MIPI0.D0_P
- SOM2001 pad 121: unconnected-(SOM2001C-MIPI0_D1_N-Pad121) -> /CM5/MIPI0.D1_N
- SOM2001 pad 123: unconnected-(SOM2001C-MIPI0_D1_P-Pad123) -> /CM5/MIPI0.D1_P
- SOM2001 pad 127: unconnected-(SOM2001C-MIPI0_C_N-Pad127) -> /CM5/MIPI0.CLK_N
- SOM2001 pad 128: unconnected-(SOM2001A-USB3-0-RX_N-Pad128) -> /CM5/USB3_0.RX_N
- SOM2001 pad 129: unconnected-(SOM2001C-MIPI0_C_P-Pad129) -> /CM5/MIPI0.CLK_P
- SOM2001 pad 130: unconnected-(SOM2001A-USB3-0-RX_P-Pad130) -> /CM5/USB3_0.RX_P
- SOM2001 pad 133: unconnected-(SOM2001C-MIPI0_D2_N-Pad133) -> /CM5/MIPI0.D2_N
- SOM2001 pad 134: unconnected-(SOM2001A-USB3-0-D_P-Pad134) -> /CM5/USB3_0.DP
- SOM2001 pad 135: unconnected-(SOM2001C-MIPI0_D2_P-Pad135) -> /CM5/MIPI0.D2_P
- SOM2001 pad 136: unconnected-(SOM2001A-USB3-0-D_N-Pad136) -> /CM5/USB3_0.DN
- SOM2001 pad 139: unconnected-(SOM2001C-MIPI0_D3_N-Pad139) -> /CM5/MIPI0.D3_N
- SOM2001 pad 140: unconnected-(SOM2001A-USB3-0-TX_N-Pad140) -> /CM5/USB3_0.TX_N
- SOM2001 pad 141: unconnected-(SOM2001C-MIPI0_D3_P-Pad141) -> /CM5/MIPI0.D3_P
- SOM2001 pad 142: unconnected-(SOM2001A-USB3-0-TX_P-Pad142) -> /CM5/USB3_0.TX_P
- SOM2001 pad 157: unconnected-(SOM2001A-USB3-1-RX_N-Pad157) -> /CM5/USB3_1.RX_N
- SOM2001 pad 159: unconnected-(SOM2001A-USB3-1-RX_P-Pad159) -> /CM5/USB3_1.RX_P
- SOM2001 pad 16: unconnected-(SOM2001D-FAN_TACHO-Pad16) -> /CM5/FAN_TACHO
- SOM2001 pad 163: unconnected-(SOM2001A-USB3-1-D_P-Pad163) -> /CM5/USB3_1.DP
- SOM2001 pad 165: unconnected-(SOM2001A-USB3-1-D_N-Pad165) -> /CM5/USB3_1.DN
- SOM2001 pad 169: unconnected-(SOM2001A-USB3-1-TX_N-Pad169) -> /CM5/USB3_1.TX_N
- SOM2001 pad 171: unconnected-(SOM2001A-USB3-1-TX_P-Pad171) -> /CM5/USB3_1.TX_P
- SOM2001 pad 175: unconnected-(SOM2001C-MIPI1_D0_N-Pad175) -> /CM5/MIPI1.D0_N
- SOM2001 pad 177: unconnected-(SOM2001C-MIPI1_D0_P-Pad177) -> /CM5/MIPI1.D0_P
- SOM2001 pad 18: unconnected-(SOM2001B-ETH_SYNC_OUT-Pad18) -> /CM5/ETH_SYNC
- SOM2001 pad 181: unconnected-(SOM2001C-MIPI1_D1_N-Pad181) -> /CM5/MIPI1.D1_N
- SOM2001 pad 183: unconnected-(SOM2001C-MIPI1_D1_P-Pad183) -> /CM5/MIPI1.D1_P
- SOM2001 pad 187: unconnected-(SOM2001C-MIPI1_C_N-Pad187) -> /CM5/MIPI1.CLK_N
- SOM2001 pad 189: unconnected-(SOM2001C-MIPI1_C_P-Pad189) -> /CM5/MIPI1.CLK_P
- SOM2001 pad 19: unconnected-(SOM2001D-FAN_PWM-Pad19) -> /CM5/FAN_PWM
- SOM2001 pad 193: unconnected-(SOM2001C-MIPI1_D2_N-Pad193) -> /CM5/MIPI1.D2_N
- SOM2001 pad 194: unconnected-(SOM2001C-MIPI1_D3_N-Pad194) -> /CM5/MIPI1.D3_N
- SOM2001 pad 195: unconnected-(SOM2001C-MIPI1_D2_P-Pad195) -> /CM5/MIPI1.D2_P
- SOM2001 pad 196: unconnected-(SOM2001C-MIPI1_D3_P-Pad196) -> /CM5/MIPI1.D3_P
- SOM2001 pad 35: unconnected-(SOM2001A-GPIO1_ID_SC-Pad35) -> /CM5/I2C1.SCL
- SOM2001 pad 36: unconnected-(SOM2001A-GPIO0_ID_SD-Pad36) -> /CM5/I2C1.SDA
- SOM2001 pad 80: unconnected-(SOM2001C-SCL0-Pad80) -> /CM5/I2C0.SCL
- SOM2001 pad 82: unconnected-(SOM2001C-SDA0-Pad82) -> /CM5/I2C0.SDA
- SOM2001 pad 94: /CM5/USB.CC1 -> /CM5/USB2_DEV.CC1
- SOM2001 pad 96: /CM5/USB.CC2 -> /CM5/USB2_DEV.CC2
- SOM2001 pad 97: unconnected-(SOM2001C-CAM_GPIO0-Pad97) -> /CM5/CAM_GPIO0
- U303 pad 1: +3V3 -> +3V3_PCIE
- U303 pad 113: +3V3 -> +3V3_PCIE
- U303 pad 15: +3V3 -> +3V3_PCIE
- U303 pad 49: +3V3 -> +3V3_PCIE
- U303 pad 64: +3V3 -> +3V3_PCIE
- U303 pad 79: +3V3 -> +3V3_PCIE
- U303 pad 8: +3V3 -> +3V3_PCIE
- U303 pad 82: +3V3 -> +3V3_PCIE
- U303 pad 84: +3V3 -> +3V3_PCIE
- U303 pad 96: +3V3 -> +3V3_PCIE
- U5001 pad 39: +3V3 -> +3V3_PCIE
- U5001 pad 65: +3V3 -> +3V3_PCIE
- U8001 pad 9: +3V3 -> +3V3_PCIE
Other:
- outline, holes or cut-outs redrawn
