File: pcbs/jabr-control-v1/m-2-e-key.kicad_sch (KiCad schematic)
At the start: 12 parts, among them J4001 MDT320E0X001, J401 U.FL-R-SMT-K_895, J402 U.FL-R-SMT-K_895, Y401 ASEK-32.768KHZ-LRT

Commit message: Schematic nearing completion, need to do GPIO and PHY decouplings caps
Parts:
- AE401, AE402: symbol Device:Antenna_Shield -> RF-CONN:EMPCB.SMAFSTJ.B.HT
Connections:
- net USB.DN renamed DN
- net USB.DP renamed DP
- net ~{BT_DISABLE} renamed BT_EN
- net ~{WL_DISABLE} renamed WL_EN
Other:
- note added: "M.2 E-Key"
- moved on the sheet: R404
